Commit message: changed models

File: src/xarm_ros/camera.urdf (robot description, URDF)
Before this commit: robot arm_camera, 1 links, 0 joints
Links:
- added link camera_optical_frame
Joints:
- added joint camera_optical_joint: type fixed, parent camera_link, child camera_optical_frame, origin xyz=0 0 0 rpy=-1.5708 0 -1.5708

File: src/xarm_ros/xarm_description/urdf/camera/realsense_d435i.urdf.xacro (robot description, xacro)
@@ -36,5 +36,5 @@
         <child link="${prefix}camera_link" />
         <!-- Камера дивиться вперед, трохи вниз (20 градусів) -->
-        <origin xyz="0.0 0.0 0.0" rpy="0 0.349 0" />
+        <origin xyz="0.0 0.0 0.0" rpy="0 1.047 0" />
       </joint>
       <joint name="${prefix}camera_depth_joint" type="fixed">

File: src/xarm_ros/xarm_description/urdf/camera/static_camera_on_base.urdf.xacro (robot description, xacro)
@@ -47,5 +47,5 @@
         - yaw=0: без обертання
       -->
-      <origin xyz="0.0 0.0 0.0" rpy="0 0 0" />
+      <origin xyz="0.0 -0.3 0.6" rpy="0 1.047 0.349" />
     </joint>
     <!-- Optical frames для камери (потрібні для ROS topics) -->
