Commit message: yolo

File: src/xarm_ros/xarm_description/urdf/camera/static_camera_on_base.urdf.xacro (robot description, xacro)
@@ -47,5 +47,5 @@
         - yaw=0: без обертання
       -->
-      <origin xyz="0.0 -0.3 0.6" rpy="0 1.047 0.349" />
+      <origin xyz="-0.1 -0.5 0.4" rpy="0 0.4 0.6" />
     </joint>
     <!-- Optical frames для камери (потрібні для ROS topics) -->
